File: 5V_Non_Iso.sch (KiCad schematic (older format))
At the start: 5 parts, among them U13 TSR_1-2450

Commit message: added filters
Changed lines of the file:
@@
 $Descr A4 11693 8268
 encoding utf-8
-Sheet 18 19
+Sheet 18 31
 Title ""
 Date ""
@@
 AR Path="/60A3C1C6/608274F5" Ref="U13"  Part="1"
 AR Path="/60A3C1D7/608274F5" Ref="U14"  Part="1"
-F 0 "U13" H 4400 2867 50  0000 C CNN
+F 0 "U14" H 4400 2867 50  0000 C CNN
 F 1 "TSR_1-2450" H 4400 2776 50  0000 C CNN
 F 2 "Converter_DCDC:Converter_DCDC_TRACO_TSR-1_THT" H 4400 2350 50  0001 L CIN
@@
 AR Path="/60A3C1C6/6082750E" Ref="C50"  Part="1"
 AR Path="/60A3C1D7/6082750E" Ref="C54"  Part="1"
-F 0 "C50" H 2768 2646 50  0000 L CNN
+F 0 "C54" H 2768 2646 50  0000 L CNN
 F 1 "CP" H 2768 2555 50  0000 L CNN
 F 2 "Capacitor_THT:CP_Radial_D6.3mm_P2.50mm" H 2688 2450 50  0001 C CNN
@@
 AR Path="/60A3C1C6/60827514" Ref="C51"  Part="1"
 AR Path="/60A3C1D7/60827514" Ref="C55"  Part="1"
-F 0 "C51" H 3415 2646 50  0000 L CNN
+F 0 "C55" H 3415 2646 50  0000 L CNN
 F 1 "100n" H 3415 2555 50  0000 L CNN
 F 2 "Capacitor_SMD:C_0603_1608Metric" H 3338 2450 50  0001 C CNN
@@
 AR Path="/60A3C1C6/60827533" Ref="C53"  Part="1"
 AR Path="/60A3C1D7/60827533" Ref="C57"  Part="1"
-F 0 "C53" H 5468 2646 50  0000 L CNN
+F 0 "C57" H 5468 2646 50  0000 L CNN
 F 1 "CP" H 5468 2555 50  0000 L CNN
 F 2 "Capacitor_THT:CP_Radial_D6.3mm_P2.50mm" H 5388 2450 50  0001 C CNN
@@
 AR Path="/60A3C1C6/60827539" Ref="C52"  Part="1"
 AR Path="/60A3C1D7/60827539" Ref="C56"  Part="1"
-F 0 "C52" H 5015 2646 50  0000 L CNN
+F 0 "C56" H 5015 2646 50  0000 L CNN
 F 1 "100n" H 5015 2555 50  0000 L CNN
 F 2 "Capacitor_SMD:C_0603_1608Metric" H 4938 2450 50  0001 C CNN

Commit message: ready for ordering
Changed lines of the file:
@@
 $Descr A4 11693 8268
 encoding utf-8
-Sheet 18 31
+Sheet 30 31
 Title ""
 Date ""
@@
 AR Path="/60A3C1C6/608274F5" Ref="U13"  Part="1"
 AR Path="/60A3C1D7/608274F5" Ref="U14"  Part="1"
-F 0 "U14" H 4400 2867 50  0000 C CNN
+F 0 "U13" H 4400 2867 50  0000 C CNN
 F 1 "TSR_1-2450" H 4400 2776 50  0000 C CNN
 F 2 "Converter_DCDC:Converter_DCDC_TRACO_TSR-1_THT" H 4400 2350 50  0001 L CIN
@@
 AR Path="/60A3C1C6/6082750E" Ref="C50"  Part="1"
 AR Path="/60A3C1D7/6082750E" Ref="C54"  Part="1"
-F 0 "C54" H 2768 2646 50  0000 L CNN
+F 0 "C50" H 2768 2646 50  0000 L CNN
 F 1 "CP" H 2768 2555 50  0000 L CNN
 F 2 "Capacitor_THT:CP_Radial_D6.3mm_P2.50mm" H 2688 2450 50  0001 C CNN
@@
 AR Path="/60A3C1C6/60827514" Ref="C51"  Part="1"
 AR Path="/60A3C1D7/60827514" Ref="C55"  Part="1"
-F 0 "C55" H 3415 2646 50  0000 L CNN
+F 0 "C51" H 3415 2646 50  0000 L CNN
 F 1 "100n" H 3415 2555 50  0000 L CNN
 F 2 "Capacitor_SMD:C_0603_1608Metric" H 3338 2450 50  0001 C CNN
@@
 AR Path="/60A3C1C6/6082751D" Ref="#PWR087"  Part="1"
 AR Path="/60A3C1D7/6082751D" Ref="#PWR092"  Part="1"
-F 0 "#PWR092" H 2650 2550 50  0001 C CNN
+F 0 "#PWR087" H 2650 2550 50  0001 C CNN
 F 1 "GND" H 2655 2627 50  0000 C CNN
 F 2 "" H 2650 2800 50  0001 C CNN
@@
 AR Path="/60A3C1C6/60827524" Ref="#PWR088"  Part="1"
 AR Path="/60A3C1D7/60827524" Ref="#PWR093"  Part="1"
-F 0 "#PWR093" H 3300 2550 50  0001 C CNN
+F 0 "#PWR088" H 3300 2550 50  0001 C CNN
 F 1 "GND" H 3305 2627 50  0000 C CNN
 F 2 "" H 3300 2800 50  0001 C CNN
@@
 AR Path="/60A3C1C6/6082752B" Ref="#PWR089"  Part="1"
 AR Path="/60A3C1D7/6082752B" Ref="#PWR094"  Part="1"
-F 0 "#PWR094" H 4400 2500 50  0001 C CNN
+F 0 "#PWR089" H 4400 2500 50  0001 C CNN
 F 1 "GND" H 4405 2577 50  0000 C CNN
 F 2 "" H 4400 2750 50  0001 C CNN
@@
 AR Path="/60A3C1C6/60827533" Ref="C53"  Part="1"
 AR Path="/60A3C1D7/60827533" Ref="C57"  Part="1"
-F 0 "C57" H 5468 2646 50  0000 L CNN
+F 0 "C53" H 5468 2646 50  0000 L CNN
 F 1 "CP" H 5468 2555 50  0000 L CNN
 F 2 "Capacitor_THT:CP_Radial_D6.3mm_P2.50mm" H 5388 2450 50  0001 C CNN
@@
 AR Path="/60A3C1C6/60827539" Ref="C52"  Part="1"
 AR Path="/60A3C1D7/60827539" Ref="C56"  Part="1"
-F 0 "C56" H 5015 2646 50  0000 L CNN
+F 0 "C52" H 5015 2646 50  0000 L CNN
 F 1 "100n" H 5015 2555 50  0000 L CNN
 F 2 "Capacitor_SMD:C_0603_1608Metric" H 4938 2450 50  0001 C CNN
@@
 AR Path="/60A3C1C6/60827545" Ref="#PWR090"  Part="1"
 AR Path="/60A3C1D7/60827545" Ref="#PWR095"  Part="1"
-F 0 "#PWR095" H 4900 2550 50  0001 C CNN
+F 0 "#PWR090" H 4900 2550 50  0001 C CNN
 F 1 "GND" H 4905 2627 50  0000 C CNN
 F 2 "" H 4900 2800 50  0001 C CNN
@@
 AR Path="/60A3C1C6/6082754C" Ref="#PWR091"  Part="1"
 AR Path="/60A3C1D7/6082754C" Ref="#PWR096"  Part="1"
-F 0 "#PWR096" H 5350 2550 50  0001 C CNN
+F 0 "#PWR091" H 5350 2550 50  0001 C CNN
 F 1 "GND" H 5355 2627 50  0000 C CNN
 F 2 "" H 5350 2800 50  0001 C CNN
