File: AR2ISS_Isolator.sch (KiCad schematic (older format))
At the start: 21 parts, among them J1 PTT_IN, J12 Conn_01x04, J2 Conn_01x04, J3 Conn_01x04, K1 G6S-2, K2 G6S-2, SW1 SW_Push_SPDT

Commit message: added filters
Changed lines of the file:
@@
 $Descr A4 11693 8268
 encoding utf-8
-Sheet 1 19
+Sheet 1 31
 Title ""
 Date ""
@@
 AR Path="/6083EA55/608DE7E0/607F3B85" Ref="R?"  Part="1"
 AR Path="/607F3B85" Ref="R44"  Part="1"
-F 0 "R44" V 5543 3300 50  0000 C CNN
-F 1 "1k" V 5634 3300 50  0000 C CNN
+F 0 "R44" V 5650 3300 50  0000 C CNN
+F 1 "1k" V 5750 3300 50  0000 C CNN
 F 2 "Resistor_SMD:R_0603_1608Metric" V 5680 3300 50  0001 C CNN
 F 3 "~" H 5750 3300 50  0001 C CNN
@@
 AR Path="/6083EA55/608DE7E0/607F46E2" Ref="R?"  Part="1"
 AR Path="/607F46E2" Ref="R45"  Part="1"
-F 0 "R45" V 5543 3400 50  0000 C CNN
-F 1 "1k" V 5634 3400 50  0000 C CNN
+F 0 "R45" V 5650 3400 50  0000 C CNN
+F 1 "1k" V 5750 3400 50  0000 C CNN
 F 2 "Resistor_SMD:R_0603_1608Metric" V 5680 3400 50  0001 C CNN
 F 3 "~" H 5750 3400 50  0001 C CNN

Commit message: ready for ordering
Parts:
- added U15, U16, U17, U18: non_plated, AR2ISS:non_plated_3mm, symbol AR2ISS:non_plated
- R1, R2: value 10k -> 5k
Connections:
- net +5V_A: now also R2.1; no longer K1.4
- net +5V_B: now also R1.2; no longer K2.4
- net GND: now also K1.4, K2.4; no longer R1.2, R2.1
- net PTT_Main: now also R2.2; no longer R1.1
- net PTT_Sub: now also R1.1; no longer R2.2
Other:
- moved on the sheet: R1, R2
Changed lines of the file:
@@
 Wire Wire Line
 	1750 4600 3600 4600
-$Comp
-L AR2ISS:+5V_A #PWR?
-U 1 1 60A253CE
-P 2350 5900
-AR Path="/60843FDF/60A253CE" Ref="#PWR?"  Part="1"
-AR Path="/60A253CE" Ref="#PWR09"  Part="1"
-F 0 "#PWR09" H 2350 5750 50  0001 C CNN
-F 1 "+5V_A" H 2365 6073 50  0000 C CNN
-F 2 "" H 2350 5900 50  0001 C CNN
-F 3 "" H 2350 5900 50  0001 C CNN
-	1    2350 5900
-	1    0    0    -1
-$EndComp
-Wire Wire Line
-	2350 5900 2350 6050
 Wire Wire Line
 	2350 6050 2600 6050
-$Comp
-L AR2ISS:+5V_B #PWR?
-U 1 1 60A277CE
-P 3950 5900
-AR Path="/60843FDF/60A277CE" Ref="#PWR?"  Part="1"
-AR Path="/60A277CE" Ref="#PWR011"  Part="1"
-F 0 "#PWR011" H 3950 5750 50  0001 C CNN
-F 1 "+5V_B" H 3965 6073 50  0000 C CNN
-F 2 "" H 3950 5900 50  0001 C CNN
-F 3 "" H 3950 5900 50  0001 C CNN
-	1    3950 5900
-	1    0    0    -1
-$EndComp
-Wire Wire Line
-	3950 5900 3950 6050
 Wire Wire Line
 	3950 6050 4250 6050
@@
 Text Label 5000 6150 0    50   ~ 0
 PTT_Sub
-Text Label 5250 3300 2    50   ~ 0
+Text Label 4800 3300 2    50   ~ 0
 PTT_Main
-Text Label 5250 3400 2    50   ~ 0
+Text Label 4800 3400 2    50   ~ 0
 PTT_Sub
 Text Notes 700  4350 3    50   ~ 0
@@
 L AR2ISS:R R?
 U 1 1 60A5BE32
-P 5450 3750
+P 4950 3050
 AR Path="/607585FC/60A5BE32" Ref="R?"  Part="1"
 AR Path="/607F13E3/60A5BE32" Ref="R?"  Part="1"
@@
 AR Path="/6083EA55/608DE7E0/60A5BE32" Ref="R?"  Part="1"
 AR Path="/60A5BE32" Ref="R2"  Part="1"
-F 0 "R2" V 5243 3750 50  0000 C CNN
-F 1 "10k" V 5334 3750 50  0000 C CNN
-F 2 "Resistor_SMD:R_0603_1608Metric" V 5380 3750 50  0001 C CNN
-F 3 "~" H 5450 3750 50  0001 C CNN
-	1    5450 3750
-	-1   0    0    1
+F 0 "R2" V 4743 3050 50  0000 C CNN
+F 1 "5k" V 4834 3050 50  0000 C CNN
+F 2 "Resistor_SMD:R_0603_1608Metric" V 4880 3050 50  0001 C CNN
+F 3 "~" H 4950 3050 50  0001 C CNN
+	1    4950 3050
+	1    0    0    -1
 $EndComp
 $Comp
 L AR2ISS:R R?
 U 1 1 60A5D404
-P 5300 3750
+P 5100 3050
 AR Path="/607585FC/60A5D404" Ref="R?"  Part="1"
 AR Path="/607F13E3/60A5D404" Ref="R?"  Part="1"
@@
 AR Path="/6083EA55/608DE7E0/60A5D404" Ref="R?"  Part="1"
 AR Path="/60A5D404" Ref="R1"  Part="1"
-F 0 "R1" V 5093 3750 50  0000 C CNN
-F 1 "10k" V 5184 3750 50  0000 C CNN
-F 2 "Resistor_SMD:R_0603_1608Metric" V 5230 3750 50  0001 C CNN
-F 3 "~" H 5300 3750 50  0001 C CNN
-	1    5300 3750
-	1    0    0    -1
-$EndComp
-Wire Wire Line
-	5300 3600 5300 3300
-Wire Wire Line
-	5300 3300 5600 3300
-Wire Wire Line
-	5250 3300 5300 3300
-Connection ~ 5300 3300
-Wire Wire Line
-	5250 3400 5450 3400
-Wire Wire Line
-	5450 3600 5450 3400
-Connection ~ 5450 3400
-Wire Wire Line
-	5450 3400 5600 3400
-$Comp
-L power:GND #PWR013
-U 1 1 60A675E0
-P 5300 4000
-F 0 "#PWR013" H 5300 3750 50  0001 C CNN
-F 1 "GND" H 5305 3827 50  0000 C CNN
-F 2 "" H 5300 4000 50  0001 C CNN
-F 3 "" H 5300 4000 50  0001 C CNN
-	1    5300 4000
-	1    0    0    -1
-$EndComp
-Wire Wire Line
-	5300 4000 5300 3900
-$Comp
-L power:GND #PWR016
-U 1 1 60A6A7BE
-P 5450 4000
-F 0 "#PWR016" H 5450 3750 50  0001 C CNN
-F 1 "GND" H 5455 3827 50  0000 C CNN
-F 2 "" H 5450 4000 50  0001 C CNN
-F 3 "" H 5450 4000 50  0001 C CNN
-	1    5450 4000
-	1    0    0    -1
-$EndComp
-Wire Wire Line
-	5450 3900 5450 4000
+F 0 "R1" V 4893 3050 50  0000 C CNN
+F 1 "5k" V 4984 3050 50  0000 C CNN
+F 2 "Resistor_SMD:R_0603_1608Metric" V 5030 3050 50  0001 C CNN
+F 3 "~" H 5100 3050 50  0001 C CNN
+	1    5100 3050
+	-1   0    0    1
+$EndComp
+Wire Wire Line
+	5100 2800 5100 2900
+Wire Wire Line
+	4950 2900 4950 2800
 $Comp
 L Connector_Generic:Conn_01x04 J3
@@
 Wire Wire Line
 	8000 1200 8650 1200
+Wire Wire Line
+	4800 3300 4950 3300
+Wire Wire Line
+	4800 3400 5100 3400
+Wire Wire Line
+	4950 3200 4950 3300
+Connection ~ 4950 3300
+Wire Wire Line
+	5100 3200 5100 3400
+Connection ~ 5100 3400
+Wire Wire Line
+	5100 3400 5600 3400
+Wire Wire Line
+	4950 3300 5600 3300
+$Comp
+L AR2ISS:+5V_B #PWR?
+U 1 1 60A0F1CE
+P 5100 2800
+AR Path="/60843FDF/60A0F1CE" Ref="#PWR?"  Part="1"
+AR Path="/60A0F1CE" Ref="#PWR0106"  Part="1"
+F 0 "#PWR0106" H 5100 2650 50  0001 C CNN
+F 1 "+5V_B" H 5115 2973 50  0000 C CNN
+F 2 "" H 5100 2800 50  0001 C CNN
+F 3 "" H 5100 2800 50  0001 C CNN
+	1    5100 2800
+	1    0    0    -1
+$EndComp
+$Comp
+L AR2ISS:+5V_A #PWR?
+U 1 1 60A10DF7
+P 4950 2800
+AR Path="/60843FDF/60A10DF7" Ref="#PWR?"  Part="1"
+AR Path="/60A10DF7" Ref="#PWR0107"  Part="1"
+F 0 "#PWR0107" H 4950 2650 50  0001 C CNN
+F 1 "+5V_A" H 4965 2973 50  0000 C CNN
+F 2 "" H 4950 2800 50  0001 C CNN
+F 3 "" H 4950 2800 50  0001 C CNN
+	1    4950 2800
+	1    0    0    -1
+$EndComp
+$Comp
+L power:GND #PWR0108
+U 1 1 60A11D57
+P 3950 6150
+F 0 "#PWR0108" H 3950 5900 50  0001 C CNN
+F 1 "GND" H 3955 5977 50  0000 C CNN
+F 2 "" H 3950 6150 50  0001 C CNN
+F 3 "" H 3950 6150 50  0001 C CNN
+	1    3950 6150
+	1    0    0    -1
+$EndComp
+$Comp
+L power:GND #PWR0109
+U 1 1 60A130DF
+P 2350 6150
+F 0 "#PWR0109" H 2350 5900 50  0001 C CNN
+F 1 "GND" H 2355 5977 50  0000 C CNN
+F 2 "" H 2350 6150 50  0001 C CNN
+F 3 "" H 2350 6150 50  0001 C CNN
+	1    2350 6150
+	1    0    0    -1
+$EndComp
+Wire Wire Line
+	2350 6150 2350 6050
+Wire Wire Line
+	3950 6150 3950 6050
+$Comp
+L AR2ISS:non_plated U15
+U 1 1 60A2D339
+P 850 900
+F 0 "U15" H 1028 953 60  0000 L CNN
+F 1 "non_plated" H 1028 847 60  0000 L CNN
+F 2 "AR2ISS:non_plated_3mm" H 850 900 60  0001 C CNN
+F 3 "" H 850 900 60  0001 C CNN
+	1    850  900
+	1    0    0    -1
+$EndComp
+$Comp
+L AR2ISS:non_plated U16
+U 1 1 60A2DE8A
+P 850 1250
+F 0 "U16" H 1028 1303 60  0000 L CNN
+F 1 "non_plated" H 1028 1197 60  0000 L CNN
+F 2 "AR2ISS:non_plated_3mm" H 850 1250 60  0001 C CNN
+F 3 "" H 850 1250 60  0001 C CNN
+	1    850  1250
+	1    0    0    -1
+$EndComp
+$Comp
+L AR2ISS:non_plated U17
+U 1 1 60A2E46A
+P 850 1600
+F 0 "U17" H 1028 1653 60  0000 L CNN
+F 1 "non_plated" H 1028 1547 60  0000 L CNN
+F 2 "AR2ISS:non_plated_3mm" H 850 1600 60  0001 C CNN
+F 3 "" H 850 1600 60  0001 C CNN
+	1    850  1600
+	1    0    0    -1
+$EndComp
+$Comp
+L AR2ISS:non_plated U18
+U 1 1 60A2EB55
+P 850 1950
+F 0 "U18" H 1028 2003 60  0000 L CNN
+F 1 "non_plated" H 1028 1897 60  0000 L CNN
+F 2 "AR2ISS:non_plated_3mm" H 850 1950 60  0001 C CNN
+F 3 "" H 850 1950 60  0001 C CNN
+	1    850  1950
+	1    0    0    -1
+$EndComp
 $EndSCHEMATC
