File: ISO1500.sch (KiCad schematic (older format))
At the start: 3 parts, among them U5 ISO1500

Commit message: added filters
Connections:
- net A: no longer U5.12 (A)
- net B: no longer U5.13 (B)
- new net filter/A_Out: U5.12 (A)
- new net filter/B_Out: U5.13 (B)
Other:
- moved on the sheet: C21, C22, U5
Changed lines of the file:
@@
 $Descr A4 11693 8268
 encoding utf-8
-Sheet 9 19
+Sheet 13 31
 Title ""
 Date ""
@@
 L Interface_UART:ISO1500 U?
 U 1 1 6073D069
-P 5250 2200
+P 3250 3200
 AR Path="/6073D069" Ref="U?"  Part="1"
 AR Path="/6073CA49/6073D069" Ref="U?"  Part="1"
@@
 AR Path="/6083EA55/608DE7E0/608751BF/6073D069" Ref="U3"  Part="1"
 AR Path="/6083EA55/608DE7E0/6087803B/6073D069" Ref="U4"  Part="1"
-F 0 "U5" H 5250 2767 50  0000 C CNN
-F 1 "ISO1500" H 5250 2676 50  0000 C CNN
-F 2 "Package_SO:SSOP-16_3.9x4.9mm_P0.635mm" H 5250 2200 50  0001 C CNN
-F 3 "http://www.ti.com/lit/ds/symlink/iso1500.pdf" H 5250 2200 50  0001 C CNN
-	1    5250 2200
-	1    0    0    -1
-$EndComp
-Wire Wire Line
-	5650 1900 5850 1900
-Wire Wire Line
-	5850 1900 5850 1650
-Wire Wire Line
-	5850 2400 5650 2400
-Wire Wire Line
-	5850 2400 5850 2600
-Wire Wire Line
-	4600 1650 4600 1900
-Wire Wire Line
-	4600 1900 4850 1900
-Wire Wire Line
-	4600 2600 4600 2400
-Wire Wire Line
-	4600 2400 4850 2400
+F 0 "U5" H 3250 3767 50  0000 C CNN
+F 1 "ISO1500" H 3250 3676 50  0000 C CNN
+F 2 "Package_SO:SSOP-16_3.9x4.9mm_P0.635mm" H 3250 3200 50  0001 C CNN
+F 3 "http://www.ti.com/lit/ds/symlink/iso1500.pdf" H 3250 3200 50  0001 C CNN
+	1    3250 3200
+	1    0    0    -1
+$EndComp
+Wire Wire Line
+	3650 2900 3850 2900
+Wire Wire Line
+	3850 2900 3850 2650
+Wire Wire Line
+	3850 3400 3650 3400
+Wire Wire Line
+	3850 3400 3850 3600
+Wire Wire Line
+	2600 2650 2600 2900
+Wire Wire Line
+	2600 2900 2850 2900
+Wire Wire Line
+	2600 3600 2600 3400
+Wire Wire Line
+	2600 3400 2850 3400
 $Comp
 L AR2ISS:C C?
 U 1 1 60745A17
-P 6350 1350
+P 5150 1550
 AR Path="/6073CA49/60745A17" Ref="C?"  Part="1"
 AR Path="/607585FC/6075A562/60745A17" Ref="C?"  Part="1"
@@
 AR Path="/6083EA55/608DE7E0/608751BF/60745A17" Ref="C12"  Part="1"
 AR Path="/6083EA55/608DE7E0/6087803B/60745A17" Ref="C14"  Part="1"
-F 0 "C22" H 6465 1396 50  0000 L CNN
-F 1 "C" H 6465 1305 50  0000 L CNN
-F 2 "Capacitor_SMD:C_0603_1608Metric" H 6388 1200 50  0001 C CNN
-F 3 "~" H 6350 1350 50  0001 C CNN
-	1    6350 1350
-	1    0    0    -1
-$EndComp
-Wire Wire Line
-	6350 1000 6350 1200
-Wire Wire Line
-	6350 1500 6350 1650
+F 0 "C22" H 5265 1596 50  0000 L CNN
+F 1 "C" H 5265 1505 50  0000 L CNN
+F 2 "Capacitor_SMD:C_0603_1608Metric" H 5188 1400 50  0001 C CNN
+F 3 "~" H 5150 1550 50  0001 C CNN
+	1    5150 1550
+	1    0    0    -1
+$EndComp
+Wire Wire Line
+	5150 1200 5150 1400
+Wire Wire Line
+	5150 1700 5150 1850
 $Comp
 L AR2ISS:C C?
 U 1 1 607517AE
-P 4100 1400
+P 2100 2400
 AR Path="/6073CA49/607517AE" Ref="C?"  Part="1"
 AR Path="/607585FC/6075A562/607517AE" Ref="C?"  Part="1"
@@
 AR Path="/6083EA55/608DE7E0/608751BF/607517AE" Ref="C11"  Part="1"
 AR Path="/6083EA55/608DE7E0/6087803B/607517AE" Ref="C13"  Part="1"
-F 0 "C21" H 4215 1446 50  0000 L CNN
-F 1 "C" H 4215 1355 50  0000 L CNN
-F 2 "Capacitor_SMD:C_0603_1608Metric" H 4138 1250 50  0001 C CNN
-F 3 "~" H 4100 1400 50  0001 C CNN
-	1    4100 1400
-	1    0    0    -1
-$EndComp
-Wire Wire Line
-	4100 1050 4100 1250
-Wire Wire Line
-	4100 1550 4100 1700
-Wire Wire Line
-	4750 2000 4850 2000
-Wire Wire Line
-	4750 2300 4850 2300
-Text HLabel 4750 2000 0    50   Output ~ 0
+F 0 "C21" H 2215 2446 50  0000 L CNN
+F 1 "C" H 2215 2355 50  0000 L CNN
+F 2 "Capacitor_SMD:C_0603_1608Metric" H 2138 2250 50  0001 C CNN
+F 3 "~" H 2100 2400 50  0001 C CNN
+	1    2100 2400
+	1    0    0    -1
+$EndComp
+Wire Wire Line
+	2100 2050 2100 2250
+Wire Wire Line
+	2100 2550 2100 2700
+Wire Wire Line
+	2750 3000 2850 3000
+Wire Wire Line
+	2750 3300 2850 3300
+Text HLabel 2750 3000 0    50   Output ~ 0
 R
-Text HLabel 4750 2300 0    50   Input ~ 0
+Text HLabel 2750 3300 0    50   Input ~ 0
 D
 Wire Wire Line
-	4850 2100 4450 2100
-Wire Wire Line
-	4450 2100 4450 2150
-Wire Wire Line
-	4450 2200 4850 2200
-Text HLabel 4400 2150 0    50   Input ~ 0
+	2850 3100 2450 3100
+Wire Wire Line
+	2450 3100 2450 3150
+Wire Wire Line
+	2450 3200 2850 3200
+Text HLabel 2400 3150 0    50   Input ~ 0
 DE
 Wire Wire Line
-	4450 2150 4400 2150
-Connection ~ 4450 2150
-Wire Wire Line
-	4450 2150 4450 2200
-Wire Wire Line
-	5750 2100 5650 2100
-Wire Wire Line
-	5750 2200 5650 2200
-Text HLabel 5750 2100 2    50   Output ~ 0
+	2450 3150 2400 3150
+Connection ~ 2450 3150
+Wire Wire Line
+	2450 3150 2450 3200
+Text HLabel 4950 2950 2    50   Output ~ 0
 B
-Text HLabel 5750 2200 2    50   Output ~ 0
+Text HLabel 4900 3400 2    50   Output ~ 0
 A
-Text HLabel 4100 1050 1    50   Input ~ 0
+Text HLabel 2100 2050 1    50   Input ~ 0
 5V
-Text HLabel 6350 1000 1    50   Input ~ 0
+Text HLabel 5150 1200 1    50   Input ~ 0
 5V_ISO
-Text HLabel 5850 1650 1    50   Input ~ 0
+Text HLabel 3850 2650 1    50   Input ~ 0
 5V_ISO
-Text HLabel 4600 1650 1    50   Input ~ 0
+Text HLabel 2600 2650 1    50   Input ~ 0
 5V
 $Comp
 L power:GND #PWR?
 U 1 1 60751FAE
-P 4100 1700
+P 2100 2700
 AR Path="/6073CA49/60751FAE" Ref="#PWR?"  Part="1"
 AR Path="/607585FC/6075A562/60751FAE" Ref="#PWR?"  Part="1"
@@
 AR Path="/6083EA55/608DE7E0/608751BF/60751FAE" Ref="#PWR036"  Part="1"
 AR Path="/6083EA55/608DE7E0/6087803B/60751FAE" Ref="#PWR038"  Part="1"
-F 0 "#PWR058" H 4100 1450 50  0001 C CNN
-F 1 "GND" H 4105 1527 50  0000 C CNN
-F 2 "" H 4100 1700 50  0001 C CNN
-F 3 "" H 4100 1700 50  0001 C CNN
-	1    4100 1700
+F 0 "#PWR052" H 2100 2450 50  0001 C CNN
+F 1 "GND" H 2105 2527 50  0000 C CNN
+F 2 "" H 2100 2700 50  0001 C CNN
+F 3 "" H 2100 2700 50  0001 C CNN
+	1    2100 2700
 	1    0    0    -1
 $EndComp
@@
 L power:GND #PWR?
 U 1 1 6073D1FE
-P 4600 2600
+P 2600 3600
 AR Path="/6073CA49/6073D1FE" Ref="#PWR?"  Part="1"
 AR Path="/607585FC/6075A562/6073D1FE" Ref="#PWR?"  Part="1"
@@
 AR Path="/6083EA55/608DE7E0/608751BF/6073D1FE" Ref="#PWR037"  Part="1"
 AR Path="/6083EA55/608DE7E0/6087803B/6073D1FE" Ref="#PWR039"  Part="1"
-F 0 "#PWR059" H 4600 2350 50  0001 C CNN
-F 1 "GND" H 4605 2427 50  0000 C CNN
-F 2 "" H 4600 2600 50  0001 C CNN
-F 3 "" H 4600 2600 50  0001 C CNN
-	1    4600 2600
-	1    0    0    -1
-$EndComp
-Text HLabel 6350 1650 3    50   Input ~ 0
+F 0 "#PWR053" H 2600 3350 50  0001 C CNN
+F 1 "GND" H 2605 3427 50  0000 C CNN
+F 2 "" H 2600 3600 50  0001 C CNN
+F 3 "" H 2600 3600 50  0001 C CNN
+	1    2600 3600
+	1    0    0    -1
+$EndComp
+Text HLabel 5150 1850 3    50   Input ~ 0
 GND_ISO
-Text HLabel 5850 2600 3    50   Input ~ 0
+Text HLabel 3850 3600 3    50   Input ~ 0
 GND_ISO
+$Sheet
+S 4150 2850 600  650
+U 6091A70E
+F0 "filter" 50
+F1 "filter.sch" 50
+F2 "A" I R 4750 3400 50
+F3 "B" I R 4750 2950 50
+F4 "A_Out" I L 4150 3200 50
+F5 "B_Out" I L 4150 3100 50
+F6 "GND" I L 4150 3400 50
+$EndSheet
+Wire Wire Line
+	4750 2950 4950 2950
+Wire Wire Line
+	4750 3400 4900 3400
+Wire Wire Line
+	3650 3100 4150 3100
+Wire Wire Line
+	3650 3200 4150 3200
+Wire Wire Line
+	4150 3400 3850 3400
+Connection ~ 3850 3400
 $EndSCHEMATC

Commit message: ready for ordering
Parts:
- removed C21: C, Capacitor_SMD:C_0603_1608Metric, symbol AR2ISS:C
- removed U5: ISO1500, Package_SO:SSOP-16_3.9x4.9mm_P0.635mm, symbol Interface_UART:ISO1500
- added U7: SP3485, Package_SO:SOIC-8_3.9x4.9mm_P1.27mm, symbol AR2ISS:SP3485
- C22: value C -> 100n
Connections:
- net 5V_ISO: now also U7.8 (VCC)
- net D: now also U7.4 (DI)
- net DE: now also U7.2 (~RE~), U7.3 (DE)
- net GND_ISO: now also U7.5 (GND)
- net R: now also U7.1 (RO)
- net filter/A_Out: now also U7.7 (B)
- net filter/B_Out: now also U7.6 (A)
Other:
- moved on the sheet: C24
