File: IsolatorGroup.sch (KiCad schematic (older format))
At the start: 14 parts, among them J6 RJ45_LED

Commit message: added filters
Connections:
- net 5V: now also R9.1; no longer R10.1
- net GND: now also R10.1; no longer R9.1
Changed lines of the file:
@@
 $Descr A4 11693 8268
 encoding utf-8
-Sheet 8 19
+Sheet 12 31
 Title ""
 Date ""
@@
 Wire Wire Line
 	4450 3750 4550 3750
-Text HLabel 4750 3500 0    50   Input ~ 0
+Text HLabel 4750 2600 0    50   Input ~ 0
 TX
 Text HLabel 4750 4300 0    50   Input ~ 0
@@
 Wire Wire Line
 	4750 2600 4950 2600
-Text HLabel 4750 2600 0    50   Output ~ 0
+Text HLabel 4750 3500 0    50   Output ~ 0
 RX
 Wire Wire Line
@@
 L power:GND #PWR?
 U 1 1 60781A82
-P 4450 2950
+P 4450 3750
 AR Path="/607585FC/60781A82" Ref="#PWR?"  Part="1"
 AR Path="/607F13E3/60781A82" Ref="#PWR?"  Part="1"
@@
 AR Path="/6083EA55/608421F3/60781A82" Ref="#PWR?"  Part="1"
 AR Path="/6083EA55/608DE7E0/60781A82" Ref="#PWR020"  Part="1"
-F 0 "#PWR040" H 4450 2700 50  0001 C CNN
-F 1 "GND" H 4455 2777 50  0000 C CNN
-F 2 "" H 4450 2950 50  0001 C CNN
-F 3 "" H 4450 2950 50  0001 C CNN
-	1    4450 2950
+F 0 "#PWR040" H 4450 3500 50  0001 C CNN
+F 1 "GND" H 4455 3577 50  0000 C CNN
+F 2 "" H 4450 3750 50  0001 C CNN
+F 3 "" H 4450 3750 50  0001 C CNN
+	1    4450 3750
 	1    0    0    -1
 $EndComp
@@
 	6300 1350 6350 1350
 Connection ~ 6350 1350
-Text HLabel 4450 3750 0    50   Input ~ 0
+Text HLabel 4450 2950 0    50   Input ~ 0
 5V
 Text HLabel 4450 4550 0    50   Input ~ 0

Commit message: ready for ordering
Parts:
- added C11, C13, C25, C27: 100n, Capacitor_SMD:C_0603_1608Metric, symbol AR2ISS:C
- added U6: Si8641BA-C-IU, Package_SO:QSOP-16_3.9x4.9mm_P0.635mm, symbol Isolator:Si8641BA-B-IU
Connections:
- net 5V: now also C11.1, C25.1, U6.1 (VDD1), U6.7 (EN1); no longer R11.1, R12.1, R9.1
- net 5V_ISO: now also R11.1, R12.1, R9.1, C13.1, C27.1, U6.10 (EN2), U6.16 (VDD2)
- net GND: now also C11.2, C25.2, U6.2 (GND1), U6.8 (GND1); no longer R10.1
- net GND_ISO: now also R10.1, C13.2, C27.2, U6.15 (GND2), U6.9 (GND2)
- net PTT_Main: now also U6.4 (A2)
- net PTT_Sub: now also U6.5 (A3)
- net RX: now also U6.6 (A4)
- net RX/D: now also U6.14 (B1)
- net TX: now also U6.3 (A1)
- net TX/R: now also U6.11 (B4)
- new net PTT_Main/D: U6.13 (B2)
- new net PTT_Sub/D: U6.12 (B3)
