File: AR2ISS_Isolator.kicad_pcb (KiCad board)
At the start: 2 copper layers, 160 x 100 mm, 165 parts, among them J1 PTT_IN, J10 Conn_01x02, J11 Conn_01x02, J12 Conn_01x04, J2 Conn_01x04, J3 Conn_01x04, J4 Conn_02x03_Odd_Even, J5 RJ45_LED, J6 RJ45_LED, J7 RJ45_LED, J8 Conn_01x02, J9 Conn_01x02, K1 G6S-2, K2 G6S-2, SW1 SW_Push_SPDT, U1 ISO1500, U10 SN75176AD, U11 SN75176AD, U12 SN75176AD, U13 TSR_1-2450, U14 TSR_1-2450, U2 ISO1500, U3 ISO1500, U4 ISO1500, U5 ISO1500, U6 ISO1500, U7 ISO1500, U8 ISO1500, U9 SN75176AD

Commit message: added filters
Parts:
- added C60: 470p, Capacitor_SMD:C_0603_1608Metric, F.Cu at (178.6, 68.0)
- added C61: 470p, Capacitor_SMD:C_0603_1608Metric, F.Cu at (178.6, 71.7)
- added C62: 1n, Capacitor_SMD:C_0603_1608Metric, F.Cu at (183.9, 67.9)
- added C63: 1n, Capacitor_SMD:C_0603_1608Metric, F.Cu at (183.9, 71.7)
- added C64: 470p, Capacitor_SMD:C_0603_1608Metric, F.Cu at (178.6, 75.7)
- added C65: 470p, Capacitor_SMD:C_0603_1608Metric, F.Cu at (178.6, 79.4)
- added C66: 1n, Capacitor_SMD:C_0603_1608Metric, F.Cu at (183.8, 75.6)
- added C67: 1n, Capacitor_SMD:C_0603_1608Metric, F.Cu at (183.8, 79.4)
- added C68: 470p, Capacitor_SMD:C_0603_1608Metric, F.Cu at (178.6, 83.5)
- added C69: 470p, Capacitor_SMD:C_0603_1608Metric, F.Cu at (178.6, 87.3)
- added C70: 1n, Capacitor_SMD:C_0603_1608Metric, F.Cu at (183.9, 83.5)
- added C71: 1n, Capacitor_SMD:C_0603_1608Metric, F.Cu at (183.9, 87.3)
- added C72: 470p, Capacitor_SMD:C_0603_1608Metric, F.Cu at (178.6, 91.5)
- added C73: 470p, Capacitor_SMD:C_0603_1608Metric, F.Cu at (178.6, 95.2)
- added C74: 1n, Capacitor_SMD:C_0603_1608Metric, F.Cu at (183.9, 91.5)
- added C75: 1n, Capacitor_SMD:C_0603_1608Metric, F.Cu at (183.9, 95.2)
- added C76: 470p, Capacitor_SMD:C_0603_1608Metric, F.Cu at (85.1, 90.1)
- added C77: 470p, Capacitor_SMD:C_0603_1608Metric, F.Cu at (85.1, 86.4)
- added C78: 1n, Capacitor_SMD:C_0603_1608Metric, F.Cu at (79.9, 90.1)
- added C79: 1n, Capacitor_SMD:C_0603_1608Metric, F.Cu at (79.9, 86.4)
- added C80: 470p, Capacitor_SMD:C_0603_1608Metric, F.Cu at (85.1, 61.8)
- added C81: 470p, Capacitor_SMD:C_0603_1608Metric, F.Cu at (85.1, 58.0)
- added C82: 1n, Capacitor_SMD:C_0603_1608Metric, F.Cu at (79.9, 61.8)
- added C83: 1n, Capacitor_SMD:C_0603_1608Metric, F.Cu at (79.9, 58.0)
- added C84: 470p, Capacitor_SMD:C_0603_1608Metric, F.Cu at (85.1, 80.8)
- added C85: 470p, Capacitor_SMD:C_0603_1608Metric, F.Cu at (85.1, 77.1)
- added C86: 1n, Capacitor_SMD:C_0603_1608Metric, F.Cu at (79.9, 80.8)
- added C87: 1n, Capacitor_SMD:C_0603_1608Metric, F.Cu at (79.9, 77.1)
- added C88: 470p, Capacitor_SMD:C_0603_1608Metric, F.Cu at (85.1, 71.3)
- added C89: 470p, Capacitor_SMD:C_0603_1608Metric, F.Cu at (85.1, 67.6)
- added C90: 1n, Capacitor_SMD:C_0603_1608Metric, F.Cu at (79.9, 71.4)
- added C91: 1n, Capacitor_SMD:C_0603_1608Metric, F.Cu at (79.9, 67.6)
- added D11: PESD2CAN, Package_TO_SOT_SMD:SOT-23_Handsoldering, F.Cu at (187.6, 69.9)
- added D12: PESD2CAN, Package_TO_SOT_SMD:SOT-23_Handsoldering, F.Cu at (187.6, 77.6)
- added D13: PESD2CAN, Package_TO_SOT_SMD:SOT-23_Handsoldering, F.Cu at (187.6, 85.5)
- added D14: PESD2CAN, Package_TO_SOT_SMD:SOT-23_Handsoldering, F.Cu at (187.6, 93.5)
- added D17: PESD2CAN, Package_TO_SOT_SMD:SOT-23_Handsoldering, F.Cu at (76.1, 88.1)
- added D18: PESD2CAN, Package_TO_SOT_SMD:SOT-23_Handsoldering, F.Cu at (76.1, 59.8)
- added D19: PESD2CAN, Package_TO_SOT_SMD:SOT-23_Handsoldering, F.Cu at (76.1, 78.8)
- added D20: PESD2CAN, Package_TO_SOT_SMD:SOT-23_Handsoldering, F.Cu at (76.1, 69.4)
- added J13: Conn_01x02, Connector_PinHeader_2.54mm:PinHeader_1x02_P2.54mm_Vertical, F.Cu at (192.6, 70.9)
- added J14: Conn_01x02, Connector_PinHeader_2.54mm:PinHeader_1x02_P2.54mm_Vertical, F.Cu at (192.6, 78.6)
- added J15: Conn_01x02, Connector_PinHeader_2.54mm:PinHeader_1x02_P2.54mm_Vertical, F.Cu at (192.6, 86.5)
- added J16: Conn_01x02, Connector_PinHeader_2.54mm:PinHeader_1x02_P2.54mm_Vertical, F.Cu at (192.6, 94.5)
- added J17: Conn_01x02, Connector_PinHeader_2.54mm:PinHeader_1x02_P2.54mm_Vertical, F.Cu at (71.1, 87.1)
- added J18: Conn_01x02, Connector_PinHeader_2.54mm:PinHeader_1x02_P2.54mm_Vertical, F.Cu at (71.1, 58.8)
- added J19: Conn_01x02, Connector_PinHeader_2.54mm:PinHeader_1x02_P2.54mm_Vertical, F.Cu at (71.1, 77.8)
- added J20: Conn_01x02, Connector_PinHeader_2.54mm:PinHeader_1x02_P2.54mm_Vertical, F.Cu at (71.1, 68.4)
- added L19: 74279266, Inductor_SMD:L_0603_1608Metric, F.Cu at (182.1, 67.9)
- added L20: 74279266, Inductor_SMD:L_0603_1608Metric, F.Cu at (182.1, 71.7)
- added L21: 10u, Inductor_SMD:L_0603_1608Metric, F.Cu at (176.9, 67.9)
- added L22: 10u, Inductor_SMD:L_0603_1608Metric, F.Cu at (176.9, 71.7)
- added L23: 74279266, Inductor_SMD:L_0603_1608Metric, F.Cu at (182.1, 75.6)
- added L24: 74279266, Inductor_SMD:L_0603_1608Metric, F.Cu at (182.1, 79.4)
- added L25: 10u, Inductor_SMD:L_0603_1608Metric, F.Cu at (176.8, 75.6)
- added L26: 10u, Inductor_SMD:L_0603_1608Metric, F.Cu at (176.8, 79.4)
- added L27: 74279266, Inductor_SMD:L_0603_1608Metric, F.Cu at (182.1, 83.5)
- added L28: 74279266, Inductor_SMD:L_0603_1608Metric, F.Cu at (182.1, 87.3)
- added L29: 10u, Inductor_SMD:L_0603_1608Metric, F.Cu at (176.9, 83.5)
- added L30: 10u, Inductor_SMD:L_0603_1608Metric, F.Cu at (176.9, 87.3)
- added L31: 74279266, Inductor_SMD:L_0603_1608Metric, F.Cu at (182.1, 91.5)
- added L32: 74279266, Inductor_SMD:L_0603_1608Metric, F.Cu at (182.1, 95.2)
- added L33: 10u, Inductor_SMD:L_0603_1608Metric, F.Cu at (176.9, 91.5)
- added L34: 10u, Inductor_SMD:L_0603_1608Metric, F.Cu at (176.9, 95.2)
- added L35: 74279266, Inductor_SMD:L_0603_1608Metric, F.Cu at (81.6, 90.1)
- added L36: 74279266, Inductor_SMD:L_0603_1608Metric, F.Cu at (81.6, 86.4)
- added L37: 10u, Inductor_SMD:L_0603_1608Metric, F.Cu at (86.9, 90.1)
- added L38: 10u, Inductor_SMD:L_0603_1608Metric, F.Cu at (86.9, 86.4)
- added L39: 74279266, Inductor_SMD:L_0603_1608Metric, F.Cu at (81.6, 61.8)
- added L40: 74279266, Inductor_SMD:L_0603_1608Metric, F.Cu at (81.6, 58.0)
- added L41: 10u, Inductor_SMD:L_0603_1608Metric, F.Cu at (86.9, 61.8)
- added L42: 10u, Inductor_SMD:L_0603_1608Metric, F.Cu at (86.9, 58.0)
- added L43: 74279266, Inductor_SMD:L_0603_1608Metric, F.Cu at (81.6, 80.8)
- added L44: 74279266, Inductor_SMD:L_0603_1608Metric, F.Cu at (81.6, 77.1)
- added L45: 10u, Inductor_SMD:L_0603_1608Metric, F.Cu at (86.9, 80.8)
- added L46: 10u, Inductor_SMD:L_0603_1608Metric, F.Cu at (86.9, 77.1)
- added L47: 74279266, Inductor_SMD:L_0603_1608Metric, F.Cu at (81.6, 71.4)
- added L48: 74279266, Inductor_SMD:L_0603_1608Metric, F.Cu at (81.6, 67.6)
- added L49: 10u, Inductor_SMD:L_0603_1608Metric, F.Cu at (86.9, 71.4)
- added L50: 10u, Inductor_SMD:L_0603_1608Metric, F.Cu at (86.9, 67.6)
- added R46: 120, Resistor_SMD:R_0603_1608Metric, F.Cu at (187.6, 72.7)
- added R47: 220, Resistor_SMD:R_0603_1608Metric, F.Cu at (180.4, 67.9)
- added R48: 220, Resistor_SMD:R_0603_1608Metric, F.Cu at (180.4, 71.7)
- added R49: 120, Resistor_SMD:R_0603_1608Metric, F.Cu at (187.6, 80.4)
- added R50: 220, Resistor_SMD:R_0603_1608Metric, F.Cu at (180.3, 75.6)
- added R51: 220, Resistor_SMD:R_0603_1608Metric, F.Cu at (180.3, 79.4)
- added R52: 120, Resistor_SMD:R_0603_1608Metric, F.Cu at (187.7, 88.2)
- added R53: 220, Resistor_SMD:R_0603_1608Metric, F.Cu at (180.4, 83.5)
- added R54: 220, Resistor_SMD:R_0603_1608Metric, F.Cu at (180.4, 87.3)
- added R55: 120, Resistor_SMD:R_0603_1608Metric, F.Cu at (187.6, 96.2)
- added R56: 220, Resistor_SMD:R_0603_1608Metric, F.Cu at (180.4, 91.5)
- added R57: 220, Resistor_SMD:R_0603_1608Metric, F.Cu at (180.4, 95.2)
- added R58: 120, Resistor_SMD:R_0603_1608Metric, F.Cu at (76.1, 85.4)
- added R59: 220, Resistor_SMD:R_0603_1608Metric, F.Cu at (83.4, 90.1)
- added R60: 220, Resistor_SMD:R_0603_1608Metric, F.Cu at (83.4, 86.4)
- added R61: 120, Resistor_SMD:R_0603_1608Metric, F.Cu at (76.1, 57.0)
- added R62: 220, Resistor_SMD:R_0603_1608Metric, F.Cu at (83.4, 61.8)
- added R63: 220, Resistor_SMD:R_0603_1608Metric, F.Cu at (83.4, 58.0)
- added R64: 120, Resistor_SMD:R_0603_1608Metric, F.Cu at (76.1, 76.1)
- added R65: 220, Resistor_SMD:R_0603_1608Metric, F.Cu at (83.4, 80.8)
- added R66: 220, Resistor_SMD:R_0603_1608Metric, F.Cu at (83.4, 77.1)
- added R67: 120, Resistor_SMD:R_0603_1608Metric, F.Cu at (76.1, 66.6)
- added R68: 220, Resistor_SMD:R_0603_1608Metric, F.Cu at (83.4, 71.4)
- added R69: 220, Resistor_SMD:R_0603_1608Metric, F.Cu at (83.4, 67.6)
- L10, L13, L14, L17, L18, L5, L6, L9: value 74279266 -> 10u
- L11, L12, L15, L16, L3, L4, L7, L8: value 10u -> 74279266
- R16, R23, R30, R37: value 221 -> 120
- R17, R24, R31, R38: value 221 -> 220
- R18, R25, R32, R39: value 120 -> 220
- moved R24 287.2 mm to (351.7, 126.6)
- moved L7 286.4 mm to (349.9, 126.6)
- moved L8 286.3 mm to (349.9, 122.9)
- moved L9 284.7 mm to (355.2, 126.6), turned to 270 degrees
- moved C35 284.7 mm to (353.4, 126.6)
- moved C36 284.6 mm to (353.4, 122.9)
- moved L10 284.6 mm to (355.2, 122.9), turned to 90 degrees
- moved C37 281.3 mm to (348.2, 126.6)
- moved C38 281.2 mm to (348.2, 122.9)
- moved R23 278.3 mm to (344.4, 121.9), turned to 180 degrees
- moved R25 273.8 mm to (351.7, 122.9), turned to 270 degrees
- moved D8 270.4 mm to (344.4, 124.6), turned to 0 degrees
- moved J9 260.4 mm to (339.4, 123.6), turned to 0 degrees
- moved R38 237.4 mm to (297.4, 144.5)
- moved L15 236.4 mm to (295.6, 144.5)
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Connections:
- C30 pad 2: GND -> /SignalsToSlave/IsolatorGroup_B/GND_ISO
- C31 pad 2: GND -> /SignalsToSlave/IsolatorGroup_B/GND_ISO
- C32 pad 2: GND -> /SignalsToSlave/IsolatorGroup_B/GND_ISO
- C33 pad 2: GND -> /SignalsToSlave/IsolatorGroup_B/GND_ISO
- C34 pad 1: /MasterInput/RS485Tranceiver1/MODE -> /MasterInput/RS485Tranceiver2/MODE
- C35 pad 2: GND -> /SignalsToSlave/IsolatorGroup_B/GND_ISO
- C36 pad 2: GND -> /SignalsToSlave/IsolatorGroup_B/GND_ISO
- C37 pad 2: GND -> /SignalsToSlave/IsolatorGroup_B/GND_ISO
- C38 pad 2: GND -> /SignalsToSlave/IsolatorGroup_B/GND_ISO
- C39 pad 1: /MasterInput/RS485Tranceiver3/MODE -> /MasterInput/RS485Tranceiver4/MODE
- C40 pad 2: GND -> /SignalsToSlave/IsolatorGroup_B/GND_ISO
- C41 pad 2: GND -> /SignalsToSlave/IsolatorGroup_B/GND_ISO
- C42 pad 2: GND -> /SignalsToSlave/IsolatorGroup_B/GND_ISO
- C43 pad 2: GND -> /SignalsToSlave/IsolatorGroup_B/GND_ISO
- C44 pad 1: /MasterInput/RS485Tranceiver1/MODE -> /MasterInput/RS485Tranceiver2/MODE
- C45 pad 2: GND -> /SignalsToSlave/IsolatorGroup_B/GND_ISO
- C46 pad 2: GND -> /SignalsToSlave/IsolatorGroup_B/GND_ISO
- C47 pad 2: GND -> /SignalsToSlave/IsolatorGroup_B/GND_ISO
- C48 pad 2: GND -> /SignalsToSlave/IsolatorGroup_B/GND_ISO
- C49 pad 1: /MasterInput/RS485Tranceiver3/MODE -> /MasterInput/RS485Tranceiver4/MODE
- D10 pad 1: Net-(D10-Pad1) -> /SignalsToSlave/IsolatorGroup_B/PTT_Sub/B
- D10 pad 2: Net-(D10-Pad2) -> /SignalsToSlave/IsolatorGroup_B/PTT_Sub/A
- D10 pad 3: GND -> /SignalsToSlave/IsolatorGroup_B/GND_ISO
- D7 pad 1: Net-(D7-Pad1) -> /SignalsToSlave/IsolatorGroup_B/RX/B
- D7 pad 2: Net-(D7-Pad2) -> /SignalsToSlave/IsolatorGroup_B/RX/A
- D7 pad 3: GND -> /SignalsToSlave/IsolatorGroup_B/GND_ISO
- D8 pad 1: Net-(D8-Pad1) -> /SignalsToSlave/IsolatorGroup_B/TX/B
- D8 pad 2: Net-(D8-Pad2) -> /SignalsToSlave/IsolatorGroup_B/TX/A
- D8 pad 3: GND -> /SignalsToSlave/IsolatorGroup_B/GND_ISO
- D9 pad 1: Net-(D9-Pad1) -> /SignalsToSlave/IsolatorGroup_B/PTT_Main/B
- D9 pad 2: Net-(D9-Pad2) -> /SignalsToSlave/IsolatorGroup_B/PTT_Main/A
- D9 pad 3: GND -> /SignalsToSlave/IsolatorGroup_B/GND_ISO
- J10 pad 2: Net-(D9-Pad2) -> /SignalsToSlave/IsolatorGroup_B/PTT_Main/A
- J11 pad 2: Net-(D10-Pad2) -> /SignalsToSlave/IsolatorGroup_B/PTT_Sub/A
- J8 pad 2: Net-(D7-Pad2) -> /SignalsToSlave/IsolatorGroup_B/RX/A
- J9 pad 2: Net-(D8-Pad2) -> /SignalsToSlave/IsolatorGroup_B/TX/A
- L1 pad 1: /MasterInput/RS485Tranceiver3/MODE -> /MasterInput/RS485Tranceiver4/MODE
- L10 pad 1: Net-(C36-Pad1) -> /SignalsToSlave/IsolatorGroup_B/TX/filter/B_Out
- L10 pad 2: Net-(D8-Pad2) -> Net-(C36-Pad1)
- L11 pad 1: /MasterInput/RS485Tranceiver2/B_in -> Net-(C40-Pad1)
- L11 pad 2: Net-(C40-Pad1) -> /SignalsToSlave/IsolatorGroup_B/PTT_Main/A
- L12 pad 1: /MasterInput/RS485Tranceiver2/A_in -> Net-(C41-Pad1)
- L12 pad 2: Net-(C41-Pad1) -> /SignalsToSlave/IsolatorGroup_B/PTT_Main/B
- L13 pad 1: Net-(C40-Pad1) -> /SignalsToSlave/IsolatorGroup_B/PTT_Main/filter/A_Out
- L13 pad 2: Net-(D9-Pad1) -> Net-(C40-Pad1)
- L14 pad 1: Net-(C41-Pad1) -> /SignalsToSlave/IsolatorGroup_B/PTT_Main/filter/B_Out
- L14 pad 2: Net-(D9-Pad2) -> Net-(C41-Pad1)
- L15 pad 1: /MasterInput/RS485Tranceiver3/B_in -> Net-(C45-Pad1)
- L15 pad 2: Net-(C45-Pad1) -> /SignalsToSlave/IsolatorGroup_B/PTT_Sub/A
- L16 pad 1: /MasterInput/RS485Tranceiver3/A_in -> Net-(C46-Pad1)
- L16 pad 2: Net-(C46-Pad1) -> /SignalsToSlave/IsolatorGroup_B/PTT_Sub/B
- L17 pad 1: Net-(C45-Pad1) -> /SignalsToSlave/IsolatorGroup_B/PTT_Sub/filter/A_Out
- L17 pad 2: Net-(D10-Pad1) -> Net-(C45-Pad1)
- L18 pad 1: Net-(C46-Pad1) -> /SignalsToSlave/IsolatorGroup_B/PTT_Sub/filter/B_Out
- L18 pad 2: Net-(D10-Pad2) -> Net-(C46-Pad1)
- L2 pad 1: /MasterInput/RS485Tranceiver1/MODE -> /MasterInput/RS485Tranceiver2/MODE
- L3 pad 1: /MasterInput/RS485Tranceiver1/B_in -> Net-(C30-Pad1)
- L3 pad 2: Net-(C30-Pad1) -> /SignalsToSlave/IsolatorGroup_B/RX/A
- L4 pad 1: /MasterInput/RS485Tranceiver1/A_in -> Net-(C31-Pad1)
- L4 pad 2: Net-(C31-Pad1) -> /SignalsToSlave/IsolatorGroup_B/RX/B
- L5 pad 1: Net-(C30-Pad1) -> /SignalsToSlave/IsolatorGroup_B/RX/filter/A_Out
- L5 pad 2: Net-(D7-Pad1) -> Net-(C30-Pad1)
- L6 pad 1: Net-(C31-Pad1) -> /SignalsToSlave/IsolatorGroup_B/RX/filter/B_Out
- L6 pad 2: Net-(D7-Pad2) -> Net-(C31-Pad1)
- L7 pad 1: /MasterInput/RS485Tranceiver4/B_in -> Net-(C35-Pad1)
- L7 pad 2: Net-(C35-Pad1) -> /SignalsToSlave/IsolatorGroup_B/TX/A
- L8 pad 1: /MasterInput/RS485Tranceiver4/A_in -> Net-(C36-Pad1)
- L8 pad 2: Net-(C36-Pad1) -> /SignalsToSlave/IsolatorGroup_B/TX/B
- L9 pad 1: Net-(C35-Pad1) -> /SignalsToSlave/IsolatorGroup_B/TX/filter/A_Out
- L9 pad 2: Net-(D8-Pad1) -> Net-(C35-Pad1)
- R10 pad 1: +5V_B -> GND
- R16 pad 1: Net-(C30-Pad1) -> /SignalsToSlave/IsolatorGroup_B/RX/B
- R16 pad 2: Net-(C32-Pad1) -> Net-(J8-Pad1)
- R17 pad 1: Net-(C31-Pad1) -> Net-(C30-Pad1)
- R17 pad 2: Net-(C33-Pad1) -> Net-(C32-Pad1)
- R18 pad 1: Net-(D7-Pad1) -> Net-(C31-Pad1)
- R18 pad 2: Net-(J8-Pad1) -> Net-(C33-Pad1)
- R19 pad 1: /MasterInput/RS485Tranceiver1/MODE -> /MasterInput/RS485Tranceiver2/MODE
- R19 pad 2: Net-(D7-Pad1) -> /MasterInput/RS485Tranceiver1/sheet60920273/B_Out
- R20 pad 1: Net-(D7-Pad1) -> /MasterInput/RS485Tranceiver1/sheet60920273/B_Out
- R20 pad 2: Net-(D7-Pad2) -> /MasterInput/RS485Tranceiver1/sheet60920273/A_Out
- R21 pad 1: Net-(D7-Pad2) -> /MasterInput/RS485Tranceiver1/sheet60920273/A_Out
- R22 pad 1: /MasterInput/RS485Tranceiver1/MODE -> GND
- R23 pad 1: Net-(C35-Pad1) -> /SignalsToSlave/IsolatorGroup_B/TX/B
- R23 pad 2: Net-(C37-Pad1) -> Net-(J9-Pad1)
- R24 pad 1: Net-(C36-Pad1) -> Net-(C35-Pad1)
- R24 pad 2: Net-(C38-Pad1) -> Net-(C37-Pad1)
- R25 pad 1: Net-(D8-Pad1) -> Net-(C36-Pad1)
- R25 pad 2: Net-(J9-Pad1) -> Net-(C38-Pad1)
- R26 pad 1: /MasterInput/RS485Tranceiver3/MODE -> /MasterInput/RS485Tranceiver4/MODE
- R26 pad 2: Net-(D8-Pad1) -> /MasterInput/RS485Tranceiver4/sheet60920273/B_Out
- R27 pad 1: Net-(D8-Pad1) -> /MasterInput/RS485Tranceiver4/sheet60920273/B_Out
- R27 pad 2: Net-(D8-Pad2) -> /MasterInput/RS485Tranceiver4/sheet60920273/A_Out
- R28 pad 1: Net-(D8-Pad2) -> /MasterInput/RS485Tranceiver4/sheet60920273/A_Out
- R29 pad 1: GND -> /MasterInput/RS485Tranceiver4/MODE
- R3 pad 1: GND -> +5V_A
- R30 pad 1: Net-(C40-Pad1) -> /SignalsToSlave/IsolatorGroup_B/PTT_Main/B
- R30 pad 2: Net-(C42-Pad1) -> Net-(J10-Pad1)
- R31 pad 1: Net-(C41-Pad1) -> Net-(C40-Pad1)
- R31 pad 2: Net-(C43-Pad1) -> Net-(C42-Pad1)
- R32 pad 1: Net-(D9-Pad1) -> Net-(C41-Pad1)
- R32 pad 2: Net-(J10-Pad1) -> Net-(C43-Pad1)
- R33 pad 1: /MasterInput/RS485Tranceiver1/MODE -> /MasterInput/RS485Tranceiver2/MODE
- R33 pad 2: Net-(D9-Pad1) -> /MasterInput/RS485Tranceiver2/sheet60920273/B_Out
- R34 pad 1: Net-(D9-Pad1) -> /MasterInput/RS485Tranceiver2/sheet60920273/B_Out
- R34 pad 2: Net-(D9-Pad2) -> /MasterInput/RS485Tranceiver2/sheet60920273/A_Out
- R35 pad 1: Net-(D9-Pad2) -> /MasterInput/RS485Tranceiver2/sheet60920273/A_Out
- R36 pad 1: GND -> /MasterInput/RS485Tranceiver2/MODE
- R37 pad 1: Net-(C45-Pad1) -> /SignalsToSlave/IsolatorGroup_B/PTT_Sub/B
- R37 pad 2: Net-(C47-Pad1) -> Net-(J11-Pad1)
- R38 pad 1: Net-(C46-Pad1) -> Net-(C45-Pad1)
- R38 pad 2: Net-(C48-Pad1) -> Net-(C47-Pad1)
- R39 pad 1: Net-(D10-Pad1) -> Net-(C46-Pad1)
- R39 pad 2: Net-(J11-Pad1) -> Net-(C48-Pad1)
- R4 pad 1: +5V_A -> GND
- R40 pad 1: /MasterInput/RS485Tranceiver3/MODE -> /MasterInput/RS485Tranceiver4/MODE
- R40 pad 2: Net-(D10-Pad1) -> /MasterInput/RS485Tranceiver3/sheet60920273/B_Out
- R41 pad 1: Net-(D10-Pad1) -> /MasterInput/RS485Tranceiver3/sheet60920273/B_Out
- R41 pad 2: Net-(D10-Pad2) -> /MasterInput/RS485Tranceiver3/sheet60920273/A_Out
- R42 pad 1: Net-(D10-Pad2) -> /MasterInput/RS485Tranceiver3/sheet60920273/A_Out
- R43 pad 1: /MasterInput/RS485Tranceiver3/MODE -> GND
- R9 pad 1: GND -> +5V_B
- U1 pad 12: /SignalsToSlave/IsolatorGroup_B/RX/A -> /SignalsToSlave/IsolatorGroup_B/RX/filter/A_Out
- U1 pad 13: /SignalsToSlave/IsolatorGroup_B/RX/B -> /SignalsToSlave/IsolatorGroup_B/RX/filter/B_Out
- U1 pad 3: /SignalsToSlave/B_RX -> /SignalsToSlave/B_TX
- U10 pad 1: /SignalsToSlave/B_TX -> /SignalsToSlave/B_RX
- U10 pad 3: /SignalsToSlave/B_TX -> /SignalsToSlave/B_RX
- U10 pad 6: Net-(D8-Pad2) -> /MasterInput/RS485Tranceiver4/sheet60920273/A_Out
- U10 pad 7: Net-(D8-Pad1) -> /MasterInput/RS485Tranceiver4/sheet60920273/B_Out
- U10 pad 8: /MasterInput/RS485Tranceiver3/MODE -> /MasterInput/RS485Tranceiver4/MODE
- U11 pad 1: /SignalsToSlave/A_TX -> /SignalsToSlave/A_RX
- U11 pad 3: /SignalsToSlave/A_TX -> /SignalsToSlave/A_RX
- U11 pad 6: Net-(D9-Pad2) -> /MasterInput/RS485Tranceiver2/sheet60920273/A_Out
- U11 pad 7: Net-(D9-Pad1) -> /MasterInput/RS485Tranceiver2/sheet60920273/B_Out
- U11 pad 8: /MasterInput/RS485Tranceiver1/MODE -> /MasterInput/RS485Tranceiver2/MODE
- U12 pad 1: /SignalsToSlave/B_RX -> /SignalsToSlave/B_TX
- U12 pad 3: /SignalsToSlave/B_RX -> /SignalsToSlave/B_TX
- U12 pad 6: Net-(D10-Pad2) -> /MasterInput/RS485Tranceiver3/sheet60920273/A_Out
- U12 pad 7: Net-(D10-Pad1) -> /MasterInput/RS485Tranceiver3/sheet60920273/B_Out
- U12 pad 8: /MasterInput/RS485Tranceiver3/MODE -> /MasterInput/RS485Tranceiver4/MODE
- U2 pad 12: /SignalsToSlave/IsolatorGroup_B/TX/A -> /SignalsToSlave/IsolatorGroup_B/TX/filter/A_Out
- U2 pad 13: /SignalsToSlave/IsolatorGroup_B/TX/B -> /SignalsToSlave/IsolatorGroup_B/TX/filter/B_Out
- U2 pad 6: /SignalsToSlave/B_TX -> /SignalsToSlave/B_RX
- U3 pad 12: /SignalsToSlave/IsolatorGroup_B/PTT_Main/A -> /SignalsToSlave/IsolatorGroup_B/PTT_Main/filter/A_Out
- U3 pad 13: /SignalsToSlave/IsolatorGroup_B/PTT_Main/B -> /SignalsToSlave/IsolatorGroup_B/PTT_Main/filter/B_Out
- U4 pad 12: /SignalsToSlave/IsolatorGroup_B/PTT_Sub/A -> /SignalsToSlave/IsolatorGroup_B/PTT_Sub/filter/A_Out
- U4 pad 13: /SignalsToSlave/IsolatorGroup_B/PTT_Sub/B -> /SignalsToSlave/IsolatorGroup_B/PTT_Sub/filter/B_Out
- U5 pad 12: /SignalsToSlave/IsolatorGroup_A/RX/A -> /SignalsToSlave/IsolatorGroup_A/RX/filter/A_Out
- U5 pad 13: /SignalsToSlave/IsolatorGroup_A/RX/B -> /SignalsToSlave/IsolatorGroup_A/RX/filter/B_Out
- U5 pad 3: /SignalsToSlave/A_RX -> /SignalsToSlave/A_TX
- U6 pad 12: /SignalsToSlave/IsolatorGroup_A/TX/A -> /SignalsToSlave/IsolatorGroup_A/TX/filter/A_Out
- U6 pad 13: /SignalsToSlave/IsolatorGroup_A/TX/B -> /SignalsToSlave/IsolatorGroup_A/TX/filter/B_Out
- U6 pad 6: /SignalsToSlave/A_TX -> /SignalsToSlave/A_RX
- U7 pad 12: /SignalsToSlave/IsolatorGroup_A/PTT_Main/A -> /SignalsToSlave/IsolatorGroup_A/PTT_Main/filter/A_Out
- U7 pad 13: /SignalsToSlave/IsolatorGroup_A/PTT_Main/B -> /SignalsToSlave/IsolatorGroup_A/PTT_Main/filter/B_Out
- U8 pad 12: /SignalsToSlave/IsolatorGroup_A/PTT_Sub/A -> /SignalsToSlave/IsolatorGroup_A/PTT_Sub/filter/A_Out
- U8 pad 13: /SignalsToSlave/IsolatorGroup_A/PTT_Sub/B -> /SignalsToSlave/IsolatorGroup_A/PTT_Sub/filter/B_Out
- U9 pad 1: /SignalsToSlave/A_RX -> /SignalsToSlave/A_TX
- U9 pad 3: /SignalsToSlave/A_RX -> /SignalsToSlave/A_TX
- U9 pad 6: Net-(D7-Pad2) -> /MasterInput/RS485Tranceiver1/sheet60920273/A_Out
- U9 pad 7: Net-(D7-Pad1) -> /MasterInput/RS485Tranceiver1/sheet60920273/B_Out
- U9 pad 8: /MasterInput/RS485Tranceiver1/MODE -> /MasterInput/RS485Tranceiver2/MODE
Routing:
- net /MasterInput/RS485Tranceiver4/B_in: track 0.05 -> 32.0 mm
- net /MasterInput/RS485Tranceiver4/A_in: track 0.00 -> 31.4 mm
- net /MasterInput/RS485Tranceiver4/MODE: track 0.00 -> 30.7 mm
- net /MasterInput/RS485Tranceiver2/MODE: track 0.00 -> 30.7 mm
- net /MasterInput/RS485Tranceiver3/MODE: track 29.8 -> 0.00 mm
- net /SignalsToSlave/IsolatorGroup_A/5V_ISO: track 86.9 -> 112.0 mm
- net /SignalsToSlave/IsolatorGroup_B/GND_ISO: track 21.7 -> 46.6 mm, vias 26 -> 42
- net /SignalsToSlave/IsolatorGroup_A/GND_ISO: track 17.9 -> 42.7 mm, vias 36 -> 30
- net /SignalsToSlave/B_TX: track 146.0 -> 123.7 mm
- net /SignalsToSlave/B_RX: track 123.7 -> 146.0 mm
- net Net-(D8-Pad1): track 21.8 -> 0.00 mm
- net Net-(D9-Pad1): track 21.8 -> 0.00 mm
- net Net-(D7-Pad1): track 21.8 -> 0.00 mm
- net Net-(D10-Pad1): track 21.8 -> 0.00 mm
- net /MasterInput/RS485Tranceiver1/MODE: track 21.6 -> 0.00 mm
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Other:
- outline, holes or cut-outs redrawn

Commit message: updated layout
Parts:
- moved L9 179.1 mm to (176.8, 109.6), turned to 90 degrees
- moved L10 178.6 mm to (176.8, 113.4), turned to 270 degrees
- moved C35 175.6 mm to (178.6, 109.7), turned to 270 degrees
- moved C36 175.1 mm to (178.6, 113.4), turned to 90 degrees
- moved R24 172.1 mm to (180.3, 109.6), turned to 270 degrees
- moved R25 171.6 mm to (180.3, 113.4), turned to 90 degrees
- moved L7 168.7 mm to (182.1, 109.6), turned to 270 degrees
- moved L8 168.1 mm to (182.1, 113.4), turned to 90 degrees
- moved C37 165.2 mm to (183.8, 109.6), turned to 270 degrees
- moved C38 164.6 mm to (183.8, 113.4), turned to 90 degrees
- moved D8 157.3 mm to (187.6, 111.6), turned to 180 degrees
- moved R23 157.0 mm to (187.6, 114.4), turned to 0 degrees
- moved J9 147.2 mm to (192.6, 112.6), turned to 180 degrees
- moved L17 125.5 mm to (176.9, 125.5), turned to 90 degrees
- moved L18 124.6 mm to (176.9, 129.2), turned to 270 degrees
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Routing:
- net /SignalsToSlave/B_RX: track 146.0 -> 118.6 mm
- net /PTT_Main_Flt: track 120.7 -> 95.7 mm
- net +5V_B: track 234.6 -> 210.3 mm
- net /SignalsToSlave/A_TX: track 109.5 -> 85.4 mm
- net /SignalsToSlave/A_RX: track 91.0 -> 67.0 mm
- net /PTT_Sub_Flt: track 120.9 -> 96.9 mm
- net +5V_A: track 205.0 -> 181.0 mm
- net /SignalsToSlave/B_TX: track 123.7 -> 100.1 mm
- net /SignalsToSlave/IsolatorGroup_B/5V_ISO: track 99.3 -> 119.8 mm, vias 12 -> 10
- net /SignalsToSlave/IsolatorGroup_B/TX/filter/A_Out: track 0.00 -> 16.1 mm, vias 0 -> 2
- net /SignalsToSlave/IsolatorGroup_B/PTT_Sub/filter/A_Out: track 0.00 -> 15.8 mm, vias 0 -> 2
- net /SignalsToSlave/IsolatorGroup_B/PTT_Main/filter/A_Out: track 0.00 -> 15.8 mm, vias 0 -> 2
- net /SignalsToSlave/IsolatorGroup_B/RX/filter/A_Out: track 0.00 -> 15.7 mm, vias 0 -> 2
- net /SignalsToSlave/IsolatorGroup_B/PTT_Sub/filter/B_Out: track 0.00 -> 12.8 mm
- net /SignalsToSlave/IsolatorGroup_B/PTT_Main/filter/B_Out: track 0.00 -> 12.8 mm
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Other:
- outline, holes or cut-outs redrawn

Commit message: ready for ordering
Parts:
- added U15: non_plated, AR2ISS:non_plated_3mm, F.Cu at (106.0, 142.5)
- added U16: non_plated, AR2ISS:non_plated_3mm, F.Cu at (206.0, 142.5)
- added U17: non_plated, AR2ISS:non_plated_3mm, F.Cu at (106.0, 57.5)
- added U18: non_plated, AR2ISS:non_plated_3mm, F.Cu at (206.0, 57.5)
- added U19: SP3485, Package_SO:SOIC-8_3.9x4.9mm_P1.27mm, F.Cu at (171.0, 86.4)
- added U20: SP3485, Package_SO:SOIC-8_3.9x4.9mm_P1.27mm, F.Cu at (171.0, 94.0)
- C10, C11, C12, C13, C14, C21, C22, C23, C24, C25, C26, C27, C28, C7, C8, C9: value C -> 100n
- R1, R2: value 10k -> 5k
- R19, R21, R26, R28, R33, R35, R40, R42: value 10k -> NB
- R20, R27, R34, R41: value 1k -> NB
- U1, U6: value ISO1500 -> Si8641BA-B-IU; footprint Package_SO:SSOP-16_3.9x4.9mm_P0.635mm -> Package_SO:QSOP-16_3.9x4.9mm_P0.635mm
- U10, U11, U12, U9: value SN75176AD -> SP3485
- U2, U3, U4, U5, U7, U8: value ISO1500 -> SP3485; footprint Package_SO:SSOP-16_3.9x4.9mm_P0.635mm -> Package_SO:SOIC-8_3.9x4.9mm_P1.27mm
- moved U5 57.5 mm to (171.0, 128.8)
- moved C13 49.2 mm to (164.4, 77.0), turned to 180 degrees
- moved C21 42.2 mm to (159.6, 110.2)
- moved C23 42.0 mm to (164.0, 117.8), turned to 180 degrees
- moved C11 40.8 mm to (159.2, 77.2)
- moved R2 21.6 mm to (103.0, 111.0), turned to 90 degrees
- moved U8 19.4 mm to (171.0, 78.8)
- moved U7 19.1 mm to (171.0, 71.2)
- moved C7 15.8 mm to (159.6, 117.8)
- moved R6 14.3 mm to (169.4, 125.0)
- moved R5 14.2 mm to (169.4, 117.4)
- moved R4 14.0 mm to (169.4, 109.8)
- moved R3 13.9 mm to (169.4, 102.2)
- moved R9 13.7 mm to (169.4, 75.0)
- moved R10 13.6 mm to (169.4, 82.6)
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Connections:
- C11 pad 1: +5V_A -> +5V_B
- C13 pad 1: +5V_A -> /SignalsToSlave/IsolatorGroup_A/5V_ISO
- C13 pad 2: GND -> /SignalsToSlave/IsolatorGroup_A/GND_ISO
- C21 pad 1: +5V_B -> +5V_A
- C23 pad 1: +5V_B -> /SignalsToSlave/IsolatorGroup_B/5V_ISO
- C23 pad 2: GND -> /SignalsToSlave/IsolatorGroup_B/GND_ISO
- C27 pad 1: +5V_B -> /SignalsToSlave/IsolatorGroup_A/5V_ISO
- C27 pad 2: GND -> /SignalsToSlave/IsolatorGroup_A/GND_ISO
- C9 pad 1: +5V_A -> /SignalsToSlave/IsolatorGroup_B/5V_ISO
- C9 pad 2: GND -> /SignalsToSlave/IsolatorGroup_B/GND_ISO
- K1 pad 4: +5V_A -> GND
- K2 pad 4: +5V_B -> GND
- R1 pad 1: /PTT_Main -> /PTT_Sub
- R1 pad 2: GND -> +5V_B
- R10 pad 1: GND -> /SignalsToSlave/IsolatorGroup_A/GND_ISO
- R11 pad 1: +5V_B -> /SignalsToSlave/IsolatorGroup_A/5V_ISO
- R12 pad 1: +5V_B -> /SignalsToSlave/IsolatorGroup_A/5V_ISO
- R19 pad 2: /MasterInput/RS485Tranceiver1/sheet60920273/B_Out -> /MasterInput/RS485Tranceiver1/sheet60920273/A_Out
- R2 pad 1: GND -> +5V_A
- R2 pad 2: /PTT_Sub -> /PTT_Main
- R20 pad 1: /MasterInput/RS485Tranceiver1/sheet60920273/B_Out -> /MasterInput/RS485Tranceiver1/sheet60920273/A_Out
- R20 pad 2: /MasterInput/RS485Tranceiver1/sheet60920273/A_Out -> /MasterInput/RS485Tranceiver1/sheet60920273/B_Out
- R21 pad 1: /MasterInput/RS485Tranceiver1/sheet60920273/A_Out -> /MasterInput/RS485Tranceiver1/sheet60920273/B_Out
- R26 pad 2: /MasterInput/RS485Tranceiver4/sheet60920273/B_Out -> /MasterInput/RS485Tranceiver4/sheet60920273/A_Out
- R27 pad 1: /MasterInput/RS485Tranceiver4/sheet60920273/B_Out -> /MasterInput/RS485Tranceiver4/sheet60920273/A_Out
- R27 pad 2: /MasterInput/RS485Tranceiver4/sheet60920273/A_Out -> /MasterInput/RS485Tranceiver4/sheet60920273/B_Out
- R28 pad 1: /MasterInput/RS485Tranceiver4/sheet60920273/A_Out -> /MasterInput/RS485Tranceiver4/sheet60920273/B_Out
- R3 pad 1: +5V_A -> /SignalsToSlave/IsolatorGroup_B/5V_ISO
- R33 pad 2: /MasterInput/RS485Tranceiver2/sheet60920273/B_Out -> /MasterInput/RS485Tranceiver2/sheet60920273/A_Out
- R34 pad 1: /MasterInput/RS485Tranceiver2/sheet60920273/B_Out -> /MasterInput/RS485Tranceiver2/sheet60920273/A_Out
- R34 pad 2: /MasterInput/RS485Tranceiver2/sheet60920273/A_Out -> /MasterInput/RS485Tranceiver2/sheet60920273/B_Out
- R35 pad 1: /MasterInput/RS485Tranceiver2/sheet60920273/A_Out -> /MasterInput/RS485Tranceiver2/sheet60920273/B_Out
- R4 pad 1: GND -> /SignalsToSlave/IsolatorGroup_B/GND_ISO
- R40 pad 2: /MasterInput/RS485Tranceiver3/sheet60920273/B_Out -> /MasterInput/RS485Tranceiver3/sheet60920273/A_Out
- R41 pad 1: /MasterInput/RS485Tranceiver3/sheet60920273/B_Out -> /MasterInput/RS485Tranceiver3/sheet60920273/A_Out
- R41 pad 2: /MasterInput/RS485Tranceiver3/sheet60920273/A_Out -> /MasterInput/RS485Tranceiver3/sheet60920273/B_Out
- R42 pad 1: /MasterInput/RS485Tranceiver3/sheet60920273/A_Out -> /MasterInput/RS485Tranceiver3/sheet60920273/B_Out
- R5 pad 1: +5V_A -> /SignalsToSlave/IsolatorGroup_B/5V_ISO
- R6 pad 1: +5V_A -> /SignalsToSlave/IsolatorGroup_B/5V_ISO
- R9 pad 1: +5V_B -> /SignalsToSlave/IsolatorGroup_A/5V_ISO
- U1 pad 11: Net-(U1-Pad11) -> /SignalsToSlave/IsolatorGroup_B/TX/R
- U1 pad 12: /SignalsToSlave/IsolatorGroup_B/RX/filter/A_Out -> /SignalsToSlave/IsolatorGroup_B/PTT_Sub/D
- U1 pad 13: /SignalsToSlave/IsolatorGroup_B/RX/filter/B_Out -> /SignalsToSlave/IsolatorGroup_B/PTT_Main/D
- U1 pad 14: Net-(U1-Pad14) -> /SignalsToSlave/IsolatorGroup_B/RX/D
- U1 pad 4: /SignalsToSlave/IsolatorGroup_B/RX/DE -> /SignalsToSlave/IsolatorGroup_B/PTT_Main
- U1 pad 5: /SignalsToSlave/IsolatorGroup_B/RX/DE -> /SignalsToSlave/IsolatorGroup_A/PTT_Main
- U1 pad 6: /SignalsToSlave/IsolatorGroup_B/RX/D -> /SignalsToSlave/B_RX
- U1 pad 7: Net-(U1-Pad7) -> +5V_A
- U10 pad 3: /SignalsToSlave/B_RX -> /MasterInput/RS485Tranceiver4/DE1
- U10 pad 4: /MasterInput/RS485Tranceiver4/DE1 -> /SignalsToSlave/B_RX
- U11 pad 3: /SignalsToSlave/A_RX -> /MasterInput/RS485Tranceiver2/DE1
- U11 pad 4: /MasterInput/RS485Tranceiver2/DE1 -> /SignalsToSlave/A_RX
- U12 pad 3: /SignalsToSlave/B_TX -> /MasterInput/RS485Tranceiver3/DE1
- U12 pad 4: /MasterInput/RS485Tranceiver3/DE1 -> /SignalsToSlave/B_TX
- U2 pad 1: +5V_A -> /SignalsToSlave/IsolatorGroup_B/RX/R
- U2 pad 2: GND -> /SignalsToSlave/IsolatorGroup_B/RX/DE
- U2 pad 3: /SignalsToSlave/IsolatorGroup_B/TX/R -> /SignalsToSlave/IsolatorGroup_B/RX/DE
- U2 pad 4: /SignalsToSlave/IsolatorGroup_B/TX/DE -> /SignalsToSlave/IsolatorGroup_B/RX/D
- U2 pad 5: /SignalsToSlave/IsolatorGroup_B/TX/DE -> /SignalsToSlave/IsolatorGroup_B/GND_ISO
- U2 pad 6: /SignalsToSlave/B_RX -> /SignalsToSlave/IsolatorGroup_B/RX/filter/B_Out
- U2 pad 7: Net-(U2-Pad7) -> /SignalsToSlave/IsolatorGroup_B/RX/filter/A_Out
- U2 pad 8: GND -> /SignalsToSlave/IsolatorGroup_B/5V_ISO
- U3 pad 1: +5V_A -> /SignalsToSlave/IsolatorGroup_B/TX/R
- U3 pad 2: GND -> /SignalsToSlave/IsolatorGroup_B/TX/DE
- U3 pad 3: /SignalsToSlave/IsolatorGroup_B/PTT_Main/R -> /SignalsToSlave/IsolatorGroup_B/TX/DE
- U3 pad 4: /SignalsToSlave/IsolatorGroup_B/PTT_Main/DE -> /SignalsToSlave/IsolatorGroup_B/TX/D
- U3 pad 5: /SignalsToSlave/IsolatorGroup_B/PTT_Main/DE -> /SignalsToSlave/IsolatorGroup_B/GND_ISO
- U3 pad 6: /SignalsToSlave/IsolatorGroup_B/PTT_Main -> /SignalsToSlave/IsolatorGroup_B/TX/filter/B_Out
- U3 pad 7: Net-(U3-Pad7) -> /SignalsToSlave/IsolatorGroup_B/TX/filter/A_Out
- U3 pad 8: GND -> /SignalsToSlave/IsolatorGroup_B/5V_ISO
- U4 pad 1: +5V_A -> /SignalsToSlave/IsolatorGroup_B/PTT_Main/R
- U4 pad 2: GND -> /SignalsToSlave/IsolatorGroup_B/PTT_Main/DE
- U4 pad 3: /SignalsToSlave/IsolatorGroup_B/PTT_Sub/R -> /SignalsToSlave/IsolatorGroup_B/PTT_Main/DE
- U4 pad 4: /SignalsToSlave/IsolatorGroup_B/PTT_Sub/DE -> /SignalsToSlave/IsolatorGroup_B/PTT_Main/D
- U4 pad 5: /SignalsToSlave/IsolatorGroup_B/PTT_Sub/DE -> /SignalsToSlave/IsolatorGroup_B/GND_ISO
- U4 pad 6: /SignalsToSlave/IsolatorGroup_A/PTT_Main -> /SignalsToSlave/IsolatorGroup_B/PTT_Main/filter/B_Out
- U4 pad 7: Net-(U4-Pad7) -> /SignalsToSlave/IsolatorGroup_B/PTT_Main/filter/A_Out
- U4 pad 8: GND -> /SignalsToSlave/IsolatorGroup_B/5V_ISO
- U5 pad 1: +5V_B -> /SignalsToSlave/IsolatorGroup_B/PTT_Sub/R
- U5 pad 2: GND -> /SignalsToSlave/IsolatorGroup_B/PTT_Sub/DE
- U5 pad 3: /SignalsToSlave/A_TX -> /SignalsToSlave/IsolatorGroup_B/PTT_Sub/DE
- U5 pad 4: /SignalsToSlave/IsolatorGroup_A/RX/DE -> /SignalsToSlave/IsolatorGroup_B/PTT_Sub/D
- U5 pad 5: /SignalsToSlave/IsolatorGroup_A/RX/DE -> /SignalsToSlave/IsolatorGroup_B/GND_ISO
- U5 pad 6: /SignalsToSlave/IsolatorGroup_A/RX/D -> /SignalsToSlave/IsolatorGroup_B/PTT_Sub/filter/B_Out
- U5 pad 7: Net-(U5-Pad7) -> /SignalsToSlave/IsolatorGroup_B/PTT_Sub/filter/A_Out
- U5 pad 8: GND -> /SignalsToSlave/IsolatorGroup_B/5V_ISO
- U6 pad 11: Net-(U6-Pad11) -> /SignalsToSlave/IsolatorGroup_A/TX/R
- U6 pad 12: /SignalsToSlave/IsolatorGroup_A/TX/filter/A_Out -> /SignalsToSlave/IsolatorGroup_A/PTT_Sub/D
- U6 pad 13: /SignalsToSlave/IsolatorGroup_A/TX/filter/B_Out -> /SignalsToSlave/IsolatorGroup_A/PTT_Main/D
- U6 pad 14: Net-(U6-Pad14) -> /SignalsToSlave/IsolatorGroup_A/RX/D
- U6 pad 3: /SignalsToSlave/IsolatorGroup_A/TX/R -> /SignalsToSlave/A_TX
- U6 pad 4: /SignalsToSlave/IsolatorGroup_A/TX/DE -> /SignalsToSlave/IsolatorGroup_A/PTT_Main
- U6 pad 5: /SignalsToSlave/IsolatorGroup_A/TX/DE -> /SignalsToSlave/IsolatorGroup_B/PTT_Main
- U6 pad 7: Net-(U6-Pad7) -> +5V_B
- U7 pad 1: +5V_B -> /SignalsToSlave/IsolatorGroup_A/RX/R
- U7 pad 2: GND -> /SignalsToSlave/IsolatorGroup_A/RX/DE
- U7 pad 3: /SignalsToSlave/IsolatorGroup_A/PTT_Main/R -> /SignalsToSlave/IsolatorGroup_A/RX/DE
- U7 pad 4: /SignalsToSlave/IsolatorGroup_A/PTT_Main/DE -> /SignalsToSlave/IsolatorGroup_A/RX/D
- U7 pad 5: /SignalsToSlave/IsolatorGroup_A/PTT_Main/DE -> /SignalsToSlave/IsolatorGroup_A/GND_ISO
- U7 pad 6: /SignalsToSlave/IsolatorGroup_A/PTT_Main -> /SignalsToSlave/IsolatorGroup_A/RX/filter/B_Out
- U7 pad 7: Net-(U7-Pad7) -> /SignalsToSlave/IsolatorGroup_A/RX/filter/A_Out
- U7 pad 8: GND -> /SignalsToSlave/IsolatorGroup_A/5V_ISO
- U8 pad 1: +5V_B -> /SignalsToSlave/IsolatorGroup_A/TX/R
- U8 pad 2: GND -> /SignalsToSlave/IsolatorGroup_A/TX/DE
- U8 pad 3: /SignalsToSlave/IsolatorGroup_A/PTT_Sub/R -> /SignalsToSlave/IsolatorGroup_A/TX/DE
- U8 pad 4: /SignalsToSlave/IsolatorGroup_A/PTT_Sub/DE -> /SignalsToSlave/IsolatorGroup_A/TX/D
- U8 pad 5: /SignalsToSlave/IsolatorGroup_A/PTT_Sub/DE -> /SignalsToSlave/IsolatorGroup_A/GND_ISO
- U8 pad 6: /SignalsToSlave/IsolatorGroup_B/PTT_Main -> /SignalsToSlave/IsolatorGroup_A/TX/filter/B_Out
- U8 pad 7: Net-(U8-Pad7) -> /SignalsToSlave/IsolatorGroup_A/TX/filter/A_Out
- U8 pad 8: GND -> /SignalsToSlave/IsolatorGroup_A/5V_ISO
- U9 pad 3: /SignalsToSlave/A_TX -> /MasterInput/RS485Tranceiver1/DE1
- U9 pad 4: /MasterInput/RS485Tranceiver1/DE1 -> /SignalsToSlave/A_TX
Routing:
- net GND: track 97.4 -> 26.8 mm, vias 33 -> 32
- net +5V_B: track 210.3 -> 183.4 mm, vias 9 -> 4
- net /SignalsToSlave/IsolatorGroup_A/5V_ISO: track 112.0 -> 131.6 mm, vias 12 -> 13
- net /SignalsToSlave/IsolatorGroup_B/PTT_Sub/D: track 0.00 -> 19.4 mm
- net /SignalsToSlave/IsolatorGroup_B/5V_ISO: track 119.8 -> 139.0 mm, vias 10 -> 11
- net /SignalsToSlave/IsolatorGroup_A/PTT_Sub/D: track 0.00 -> 18.5 mm
- net +5V_A: track 181.0 -> 166.5 mm, vias 8 -> 5
- net /SignalsToSlave/IsolatorGroup_A/GND_ISO: track 42.7 -> 28.8 mm, vias 38 -> 32
- net /SignalsToSlave/IsolatorGroup_B/PTT_Main/D: track 0.00 -> 12.4 mm
- net /SignalsToSlave/IsolatorGroup_A/PTT_Sub/filter/A_Out: track 15.8 -> 3.84 mm, vias 2 -> 0
- net /SignalsToSlave/IsolatorGroup_A/TX/filter/A_Out: track 16.1 -> 4.09 mm, vias 2 -> 0
- net /SignalsToSlave/IsolatorGroup_A/PTT_Main/filter/A_Out: track 15.8 -> 4.00 mm, vias 2 -> 0
- net /SignalsToSlave/IsolatorGroup_B/PTT_Sub/filter/A_Out: track 15.8 -> 4.18 mm, vias 2 -> 0
- net /SignalsToSlave/IsolatorGroup_B/TX/filter/A_Out: track 16.1 -> 4.51 mm, vias 2 -> 0
- net /SignalsToSlave/IsolatorGroup_A/PTT_Main/D: track 0.00 -> 11.5 mm
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Other:
- outline, holes or cut-outs redrawn

Commit message: silkscreen
Other:
- board text added: "1"
- board text added: "12V A GND 12V B GND"
- board text added: "AR2ISS Isolator by DO4DKW"
- board text added: "Debug"
- board text added: "IN"
- board text added: "Main"
- board text added: "PTT A PTT B 12V GND"
- board text added: "PTT IN GND"
- board text added: "Rel A Rel A Rel B Rel B"
- board text added: "Sub"

Commit message: ready for jlc
Routing:
- net GND: vias 32 -> 170
- net /SignalsToSlave/IsolatorGroup_B/GND_ISO: vias 31 -> 70
- net /SignalsToSlave/IsolatorGroup_A/GND_ISO: vias 32 -> 72
Other:
- board text added: "AR2ISS Isolator by DO4DKW 2021"
- board text removed: "AR2ISS Isolator by DO4DKW"
